File: pcb/switch_matrix.kicad_sch (KiCad schematic)
At the start: 44 parts

Commit message: fix diff between updated pcb and schematic
Parts:
- added D3: ~, ComboDiode, symbol Device:D
- added S3: ~, MX, symbol Switch:SW_Push_45deg
- renumbered D9 to D10, D10 to D11, D11 to D12, D12 to D13, D13 to D14, D14 to D15, D15 to D16, D16 to D17, D17 to D18, D18 to D19, D19 to D20, D20 to D21, D21 to D22, D22 to D23, D3 to D4, D4 to D5, D5 to D6, D6 to D7, D7 to D8, D8 to D9, S9 to S10, S10 to S11, S11 to S12, S12 to S13, S13 to S14, S14 to S15, S15 to S16, S16 to S17, S17 to S18, S18 to S19, S19 to S20, S20 to S21, S21 to S22, S22 to S23, S3 to S4, S4 to S5, S5 to S6, S6 to S7, S7 to S8, S8 to S9
Connections:
- net P0: now also S3.1
- net P6: now also D3.1 (K)
- new net: D3.2 (A), S3.2

Commit message: finish pcb routing, generate fabrication file and bom
Parts:
- D1, D10, D11, D12, D13, D14, D15, D16, D17, D18, D19, D2, D20, D21, D22, D23, D3, D4, D5, D6, D7, D8, D9: footprint ComboDiode -> Diode_SMD:D_SOD-123
- S1, S10, S11, S12, S13, S14, S15, S16, S17, S18, S19, S2, S20, S21, S22, S23, S3, S4, S5, S6, S7, S8, S9: footprint MX -> (none)
Changed lines of the file:
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@@
 			)
 		)
-		(property "Footprint" "MX"
+		(property "Footprint" ""
 			(at 171.45 144.78 0)
 			(effects
@@
 			)
 		)
-		(property "Footprint" "MX"
+		(property "Footprint" ""
 			(at 222.25 43.18 0)
 			(effects
@@
 			)
 		)
-		(property "Footprint" "ComboDiode"
+		(property "Footprint" "Diode_SMD:D_SOD-123"
 			(at 97.79 76.2 0)
 			(effects
@@
 			)
 		)
-		(property "Footprint" "MX"
+		(property "Footprint" ""
 			(at 120.65 93.98 0)
 			(effects
@@
 			)
 		)
-		(property "Footprint" "ComboDiode"
+		(property "Footprint" "Diode_SMD:D_SOD-123"
 			(at 148.59 76.2 0)
 			(effects
@@
 			)
 		)
-		(property "Footprint" "ComboDiode"
+		(property "Footprint" "Diode_SMD:D_SOD-123"
 			(at 123.19 101.6 0)
 			(effects
@@
 			)
 		)
-		(property "Footprint" "MX"
+		(property "Footprint" ""
 			(at 196.85 144.78 0)
 			(effects
@@
 			)
 		)
-		(property "Footprint" "ComboDiode"
+		(property "Footprint" "Diode_SMD:D_SOD-123"
 			(at 199.39 50.8 0)
 			(effects
@@
 			)
 		)
-		(property "Footprint" "MX"
+		(property "Footprint" ""
 			(at 171.45 68.58 0)
 			(effects
@@
 			)
 		)
-		(property "Footprint" "MX"
+		(property "Footprint" ""
 			(at 120.65 68.58 0)
 			(effects
@@
 			)
 		)
-		(property "Footprint" "MX"
+		(property "Footprint" ""
 			(at 171.45 119.38 0)
 			(effects
@@
 			)
 		)
-		(property "Footprint" "ComboDiode"
+		(property "Footprint" "Diode_SMD:D_SOD-123"
 			(at 224.79 76.2 0)
 			(effects
@@
 			)
 		)
-		(property "Footprint" "MX"
+		(property "Footprint" ""
 			(at 120.65 43.18 0)
 			(effects
@@
 			)
 		)
-		(property "Footprint" "ComboDiode"
+		(property "Footprint" "Diode_SMD:D_SOD-123"
 			(at 224.79 101.6 0)
 			(effects
@@
 			)
 		)
-		(property "Footprint" "ComboDiode"
+		(property "Footprint" "Diode_SMD:D_SOD-123"
 			(at 123.19 76.2 0)
 			(effects
@@
 			)
 		)
-		(property "Footprint" "ComboDiode"
+		(property "Footprint" "Diode_SMD:D_SOD-123"
 			(at 173.99 101.6 0)
 			(effects
@@
 			)
 		)
-		(property "Footprint" "ComboDiode"
+		(property "Footprint" "Diode_SMD:D_SOD-123"
 			(at 148.59 50.8 0)
 			(effects
@@
 			)
 		)
-		(property "Footprint" "MX"
+		(property "Footprint" ""
 			(at 196.85 43.18 0)
 			(effects
@@
 			)
 		)
-		(property "Footprint" "MX"
+		(property "Footprint" ""
 			(at 222.25 93.98 0)
 			(effects
@@
 			)
 		)
-		(property "Footprint" "ComboDiode"
+		(property "Footprint" "Diode_SMD:D_SOD-123"
 			(at 173.99 50.8 0)
 			(effects
@@
 			)
 		)
-		(property "Footprint" "MX"
+		(property "Footprint" ""
 			(at 222.25 144.78 0)
 			(effects
@@
 			)
 		)
-		(property "Footprint" "MX"
+		(property "Footprint" ""
 			(at 171.45 93.98 0)
 			(effects
@@
 			)
 		)
-		(property "Footprint" "ComboDiode"
+		(property "Footprint" "Diode_SMD:D_SOD-123"
 			(at 173.99 152.4 0)
 			(effects
@@
 			)
 		)
-		(property "Footprint" "MX"
+		(property "Footprint" ""
 			(at 196.85 93.98 0)
 			(effects
@@
 			)
 		)
-		(property "Footprint" "MX"
+		(property "Footprint" ""
 			(at 171.45 43.18 0)
 			(effects
@@
 			)
 		)
-		(property "Footprint" "ComboDiode"
+		(property "Footprint" "Diode_SMD:D_SOD-123"
 			(at 97.79 50.8 0)
 			(effects
@@
 			)
 		)
-		(property "Footprint" "ComboDiode"
+		(property "Footprint" "Diode_SMD:D_SOD-123"
 			(at 199.39 152.4 0)
 			(effects
@@
 			)
 		)
-		(property "Footprint" "MX"
+		(property "Footprint" ""
 			(at 196.85 119.38 0)
 			(effects
@@
 			)
 		)
-		(property "Footprint" "MX"
+		(property "Footprint" ""
 			(at 196.85 68.58 0)
 			(effects
@@
 			)
 		)
-		(property "Footprint" "ComboDiode"
+		(property "Footprint" "Diode_SMD:D_SOD-123"
 			(at 97.79 101.6 0)
 			(effects
@@
 			)
 		)
-		(property "Footprint" "MX"
+		(property "Footprint" ""
 			(at 146.05 68.58 0)
 			(effects
@@
 			)
 		)
-		(property "Footprint" "MX"
+		(property "Footprint" ""
 			(at 95.25 43.18 0)
 			(effects
@@
 			)
 		)
-		(property "Footprint" "ComboDiode"
+		(property "Footprint" "Diode_SMD:D_SOD-123"
 			(at 224.79 152.4 0)
 			(effects
@@
 			)
 		)
-		(property "Footprint" "ComboDiode"
+		(property "Footprint" "Diode_SMD:D_SOD-123"
 			(at 173.99 76.2 0)
 			(effects
@@
 			)
 		)
-		(property "Footprint" "ComboDiode"
+		(property "Footprint" "Diode_SMD:D_SOD-123"
 			(at 199.39 127 0)
 			(effects
@@
 			)
 		)
-		(property "Footprint" "MX"
+		(property "Footprint" ""
 			(at 146.05 43.18 0)
 			(effects
@@
 			)
 		)
-		(property "Footprint" "MX"
+		(property "Footprint" ""
 			(at 222.25 68.58 0)
 			(effects
@@
 			)
 		)
-		(property "Footprint" "MX"
+		(property "Footprint" ""
 			(at 95.25 68.58 0)
 			(effects
@@
 			)
 		)
-		(property "Footprint" "ComboDiode"
+		(property "Footprint" "Diode_SMD:D_SOD-123"
 			(at 123.19 50.8 0)
 			(effects
@@
 			)
 		)
-		(property "Footprint" "ComboDiode"
+		(property "Footprint" "Diode_SMD:D_SOD-123"
 			(at 173.99 127 0)
 			(effects
@@
 			)
 		)
-		(property "Footprint" "ComboDiode"
+		(property "Footprint" "Diode_SMD:D_SOD-123"
 			(at 224.79 50.8 0)
 			(effects
@@
 			)
 		)
-		(property "Footprint" "ComboDiode"
+		(property "Footprint" "Diode_SMD:D_SOD-123"
 			(at 148.59 101.6 0)
 			(effects
@@
 			)
 		)
-		(property "Footprint" "ComboDiode"
+		(property "Footprint" "Diode_SMD:D_SOD-123"
 			(at 199.39 76.2 0)
 			(effects
@@
 			)
 		)
-		(property "Footprint" "MX"
+		(property "Footprint" ""
 			(at 146.05 93.98 0)
 			(effects
@@
 			)
 		)
-		(property "Footprint" "ComboDiode"
+		(property "Footprint" "Diode_SMD:D_SOD-123"
 			(at 199.39 101.6 0)
 			(effects
@@
 			)
 		)
-		(property "Footprint" "MX"
+		(property "Footprint" ""
 			(at 95.25 93.98 0)
 			(effects
